Commit message: Fix FK, make URDF path a variable

File: pinocchio/src/assets/parol6.urdf (robot description, URDF)
Before this commit: robot parol6, 8 links, 7 joints
Links:
- added link tcp_link
Joints:
- added joint tool_to_tcp: type fixed, parent tool, child tcp_link, origin xyz=0 0 -0.085 rpy=0 0 0

Commit message: Update URDF to match my frame assignment + add a lil benchmark for fk and jacobian calcs

File: pinocchio/src/assets/parol6.urdf (robot description, URDF)
Before this commit: robot parol6, 9 links, 8 joints
Joints:
- removed joint L1
- removed joint L2
- removed joint L3
- removed joint L4
- removed joint L5
- removed joint L6
- added joint J1: type revolute, parent base_link, child L1, origin xyz=0 0 0 rpy=0 0 0, axis 0 0 1, limit lower=-2.147 upper=2.147 effort=300 velocity=3
- added joint J2: type revolute, parent L1, child L2, origin xyz=0.0234207210610375 0 0.0 rpy=-1.5707963267949 -1.5707963267949 0, axis 0 0 1, limit lower=-0.98 upper=1 effort=300 velocity=3
- added joint J3: type revolute, parent L2, child L3, origin xyz=0.18 0 0 rpy=0 0 0, axis 0 0 1, limit lower=-2 upper=1.3 effort=300 velocity=3
- added joint J4: type revolute, parent L3, child L4, origin xyz=0.0435 0.17635 0 rpy=-1.5707963267949 0 0, axis 0 0 1, limit lower=-2 upper=2 effort=300 velocity=3
- added joint J5: type revolute, parent L4, child L5, origin xyz=0 0 0 rpy=1.5707963267949 0 0, axis 0 0 1, limit lower=-2.1 upper=2.1 effort=300 velocity=3
- added joint J6: type revolute, parent L5, child tool, origin xyz=0 0 0 rpy=-1.5707963267949 0 0, axis 0 0 1, limit lower=-3.1 upper=3.1 effort=300 velocity=3
- joint base_joint: origin xyz=0.0 0.0 0.00 rpy=0 0 0 -> xyz=0.0 0.0 0.1105 rpy=0.0 0 0
- joint tool_to_tcp: origin xyz=0 0 -0.085 rpy=0 0 0 -> xyz=0 0 0.084 rpy=0 0 -1.5707963267949

Commit message: Update joint limits in URDF

File: pinocchio/src/assets/parol6.urdf (robot description, URDF)
Before this commit: robot parol6, 9 links, 8 joints
Joints:
- joint J1: limit lower=-2.147 upper=2.147 effort=300 velocity=3 -> lower=-3.054 upper=2.880 effort=300 velocity=3
- joint J2: limit lower=-0.98 upper=1 effort=300 velocity=3 -> lower=-0.873 upper=1.484 effort=300 velocity=3
- joint J3: limit lower=-2 upper=1.3 effort=300 velocity=3 -> lower=-2.541 upper=1.222 effort=300 velocity=3
- joint J4: limit lower=-2 upper=2 effort=300 velocity=3 -> lower=-3.403 upper=1.920 effort=300 velocity=3
- joint J5: limit lower=-2.1 upper=2.1 effort=300 velocity=3 -> lower=-2.007 upper=2.007 effort=300 velocity=3

Commit message: Update TCP offset for parallel gripper

File: pinocchio/src/assets/parol6.urdf (robot description, URDF)
Before this commit: robot parol6, 9 links, 8 joints
Joints:
- joint tool_to_tcp: origin xyz=0 0 0.084 rpy=0 0 -1.5707963267949 -> xyz=0 0 0.154 rpy=0 0 -1.5707963267949
