Commit message: Add Mujoco XML + remove old DAE files

File: pinocchio/src/assets/parol6-PGripper.urdf (robot description, URDF)
Before this commit: robot parol6, 11 links, 10 joints
Links:
- link left_jaw: geometry collision mesh filename=meshes/ParallelGripper/Gripper2_Jaw.stl scale=0.01 0.01 0.01; visual mesh filename=meshes/ParallelGripper/Gripper2_Jaw.stl scale=0.01 0.01 0.01
- link right_jaw: geometry collision mesh filename=meshes/ParallelGripper/Gripper2_Jaw.stl scale=0.01 0.01 0.01; visual mesh filename=meshes/ParallelGripper/Gripper2_Jaw.stl scale=0.01 0.01 0.01
- link tool: geometry collision mesh filename=meshes/ParallelGripper/Gripper2_base_with_servo.stl scale=0.01 0.01 0.01; visual mesh filename=meshes/ParallelGripper/Gripper2_base_with_servo.stl scale=0.01 0.01 0.01
